File: hardware/32u4-programmer.sch (KiCad schematic (older format))
At the start: 42 parts

Commit message: Renamed project and updated readme.
Parts:
- U?: symbol 32u4_EEPROM:28C256 -> 32u4-programmer-rescue:28C256-32u4_EEPROM
- U?: symbol 32u4_EEPROM:28C16 -> 32u4-programmer-rescue:28C16-32u4_EEPROM
- U?: symbol 32u4_EEPROM:28C040 -> 32u4-programmer-rescue:28C040-32u4_EEPROM
Changed lines of the file:
@@
 EESchema Schematic File Version 4
+LIBS:32u4-programmer-cache
 EELAYER 26 0
 EELAYER END
@@
 	5700 6050 5950 6050
 $Comp
-L 32u4_EEPROM:28C256 U?
+L 32u4-programmer-rescue:28C256-32u4_EEPROM U?
 U 1 1 5E0D6DFC
 P 8850 4450
@@
 $EndComp
 $Comp
-L 32u4_EEPROM:28C16 U?
+L 32u4-programmer-rescue:28C16-32u4_EEPROM U?
 U 1 1 5E0DE7CC
 P 7250 4000
@@
 	3950 2800 4450 2800
 $Comp
-L 32u4_EEPROM:28C040 U?
+L 32u4-programmer-rescue:28C040-32u4_EEPROM U?
 U 1 1 5E42D5D8
 P 10400 4850
